File: PCB/hal9000mainboard.kicad_sch (KiCad schematic)
At the start: 19 parts, among them J1001 Conn_01x02, J1002 Conn_01x04, J1003 Conn_01x02, J1004 Conn_01x02, J1005 Conn_01x03, J1006 Conn_01x08, U1001 DFR0299, U1002 MOUDLE-SEEEDUINO-XIAO-ESP32C3

Commit message: adxl345 fix, renaming, and song playing
Connections:
- net +5V: now also J1006.2 (Pin_2); no longer J1006.1 (Pin_1)
- net GND: now also J1006.1 (Pin_1); no longer J1006.2 (Pin_2)
Changed lines of the file:
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@@
-	(wire
-		(pts
-			(xy 35.56 116.84) (xy 46.99 116.84)
-		)
-		(stroke
-			(width 0)
-			(type default)
-		)
-	)
 	(wire
 		(pts
@@
 	(wire
 		(pts
+			(xy 35.56 116.84) (xy 53.34 116.84)
+		)
+		(stroke
+			(width 0)
+			(type default)
+		)
+	)
+	(wire
+		(pts
 			(xy 90.17 106.68) (xy 97.79 106.68)
 		)
@@
 	(wire
 		(pts
-			(xy 46.99 116.84) (xy 46.99 119.38)
-		)
-		(stroke
-			(width 0)
-			(type default)
-		)
-	)
-	(wire
-		(pts
 			(xy 35.56 31.75) (xy 38.1 31.75)
 		)
@@
 		(pts
 			(xy 162.56 35.56) (xy 172.72 35.56)
-		)
-		(stroke
-			(width 0)
-			(type default)
-		)
-	)
-	(wire
-		(pts
-			(xy 35.56 114.3) (xy 46.99 114.3)
 		)
 		(stroke
@@
 	(symbol
 		(lib_id "power:+5V")
-		(at 46.99 114.3 0)
+		(at 53.34 116.84 0)
 		(unit 1)
 		(exclude_from_sim no)
@@
 		(fields_autoplaced yes)
 		(property "Reference" "#PWR01012"
-			(at 46.99 118.11 0)
+			(at 53.34 120.65 0)
 			(effects
 				(font
@@
 		)
 		(property "Value" "+5V"
-			(at 46.99 109.22 0)
+			(at 53.34 111.76 0)
 			(effects
 				(font
@@
 		)
 		(property "Footprint" ""
-			(at 46.99 114.3 0)
+			(at 53.34 116.84 0)
 			(effects
 				(font
@@
 		)
 		(property "Datasheet" ""
-			(at 46.99 114.3 0)
+			(at 53.34 116.84 0)
 			(effects
 				(font
@@
 		)
 		(property "Description" ""
-			(at 46.99 114.3 0)
+			(at 53.34 116.84 0)
 			(effects
 				(font
@@
 	(symbol
 		(lib_id "power:GND")
-		(at 46.99 119.38 0)
+		(at 35.56 114.3 90)
 		(unit 1)
 		(exclude_from_sim no)
@@
 		(fields_autoplaced yes)
 		(property "Reference" "#PWR01013"
-			(at 46.99 125.73 0)
+			(at 41.91 114.3 0)
 			(effects
 				(font
@@
 		)
 		(property "Value" "GND"
-			(at 46.99 124.46 0)
-			(effects
-				(font
-					(size 1.27 1.27)
-				)
+			(at 39.37 114.2999 90)
+			(effects
+				(font
+					(size 1.27 1.27)
+				)
+				(justify right)
 			)
 		)
 		(property "Footprint" ""
-			(at 46.99 119.38 0)
+			(at 35.56 114.3 0)
 			(effects
 				(font
@@
 		)
 		(property "Datasheet" ""
-			(at 46.99 119.38 0)
+			(at 35.56 114.3 0)
 			(effects
 				(font
@@
 		)
 		(property "Description" ""
-			(at 46.99 119.38 0)
-			(effects
-				(font
+			(at 35.56 114.3 0)
+			(effects
+				(font
